File: PCB/MacropadPCB.kicad_sch (KiCad schematic)
At the start: 9 parts, among them SW1 SW_Push, SW2 SW_Push, SW3 SW_Push, SW4 SW_Push, SW5 SW_Push, SW6 SW_Push, U1 XIAO-RP2040-DIP

Commit message: VERSION 3
Parts:
- removed D1, D2: SK6812MINI, LED_SMD:LED_SK6812MINI_PLCC4_3.5x3.5mm_P1.75mm, symbol LED:SK6812MINI
- added SW7: RotaryEncoder_Switch, Rotary_Encoder:RotaryEncoder_Alps_EC11E-Switch_Vertical_H20mm, symbol Device:RotaryEncoder_Switch
Connections:
- net GND: now also SW7.C, SW7.S1
- net at SW2.2: now also SW1.2, U1.5 (GPIO6/SDA); no longer U1.9 (GPIO2/SCK)
- net at SW6.2: now also U1.9 (GPIO2/SCK); no longer U1.6 (GPIO7/SCL)
- net at U1.11 (GPIO3/MOSI): now also SW7.A; no longer SW4.2
- net at SW5.2: now also U1.8 (GPIO1/RX); no longer U1.5 (GPIO6/SDA)
- net at U1.7 (GPIO0/TX): now also SW4.2
- net at U1.10 (GPIO4/MISO): now also SW7.B; no longer SW3.2
- net at U1.4 (GPIO29/ADC3/A3): now also SW7.S2
- new net: SW3.2, U1.6 (GPIO7/SCL)
Other:
- moved on the sheet: U1
